File: N39_octopus/N39_octopus.kicad_pcb (KiCad board)
At the start: 2 copper layers, 71.6 x 69.5 mm, 6 parts, among them SW1 SW_Push

Commit message: Update placements
Other:
- outline, holes or cut-outs redrawn
